File: Hardware/ts100.sch (KiCad schematic (older format))
At the start: 1 part

Commit message: hardware
Parts:
- removed U?: LM2596S-3.3_NOPB, Package_TO_SOT_SMD:TO-263-5_TabPin6, symbol KIGIT_DC-DC:LM2596S-3.3_NOPB
Changed lines of the file:
@@
 Comment4 ""
 $EndDescr
-$Comp
-L KIGIT_DC-DC:LM2596S-3.3_NOPB U?
-U 1 1 6142212F
-P 3275 2925
-F 0 "U?" H 3275 3511 60  0000 C CNN
-F 1 "LM2596S-3.3_NOPB" H 3275 3405 60  0000 C CNN
-F 2 "Package_TO_SOT_SMD:TO-263-5_TabPin6" H 3275 2865 60  0001 C CNN
-F 3 "" H 3275 2925 60  0000 C CNN
-F 4 "C90690" H 3275 2925 50  0001 C CNN "PartNum"
-	1    3275 2925
-	1    0    0    -1
-$EndComp
 $EndSCHEMATC

Commit message: parts
Parts:
- added Q?: IRF4905STRLPBF, Package_TO_SOT_SMD:TO-263-2, symbol Device:Q_PMOS_GDS
Changed lines of the file:
@@
 Comment4 ""
 $EndDescr
+$Comp
+L Device:Q_PMOS_GDS Q?
+U 1 1 61430E65
+P 2800 2750
+F 0 "Q?" H 3004 2796 50  0000 L CNN
+F 1 "IRF4905STRLPBF" H 3004 2705 50  0000 L CNN
+F 2 "Package_TO_SOT_SMD:TO-263-2" H 3000 2850 50  0001 C CNN
+F 3 "~" H 2800 2750 50  0001 C CNN
+F 4 "C2620 " H 2800 2750 50  0001 C CNN "PartNum"
+	1    2800 2750
+	1    0    0    -1
+$EndComp
 $EndSCHEMATC
