File: Hardware/ts100.sch (KiCad schematic (older format))
At the start: 1 part

Commit message: hardware
Parts:
- added C?: 10u, Capacitor_SMD:C_0805_2012Metric, symbol Device:C_Small
- added C? (x7): 0.1u, symbol Device:C_Small
- added C?: 10n, symbol Device:C_Small
- added C?: 22u, Capacitor_SMD:C_0805_2012Metric, symbol Device:C_Small
- added C?: 2.2n, symbol Device:C_Small
- added C? (x2): 22p, symbol Device:C_Small
- added D?: 1N5819, symbol Device:D_Schottky_Small_ALT
- added J?: Jack-DC, symbol Connector:Jack-DC
- added J?: Iron+, symbol Connector_Generic:Conn_01x01
- added J?: Iron-, symbol Connector_Generic:Conn_01x01
- added J?: GND, symbol Connector_Generic:Conn_01x01
- added J?: SWD, symbol Connector_Generic:Conn_02x03_Odd_Even
- added L?: 6.8u, symbol Device:L_Small
- added Q?: 2SC3356, Package_TO_SOT_SMD:SOT-23, symbol Device:Q_NPN_BEC
- added R?: 100k, symbol Device:R_Small
- added R?: 31.25k, symbol Device:R_Small
- added R? (x5): 10k, symbol Device:R_Small
- added R? (x5): R_Small, symbol Device:R_Small
- added R?: 1k, symbol Device:R_Small
- added R?: 1M, symbol Device:R_Small
- added RV?: 500k, ts100:3362P, symbol Device:R_POT_Small
- added U?: EUP3476, Package_SO:SOIC-8-1EP_3.9x4.9mm_P1.27mm_EP2.29x3mm_ThermalVias, symbol KIGIT_DC-DC:EUP3476
- added U?: 1N4728A, Diode_THT:D_DO-41_SOD81_P7.62mm_Horizontal, symbol Reference_Voltage:LM4040DBZ-8.2
- added U? (x3): AD823, Package_SO:SOP-8_3.9x4.9mm_P1.27mm, symbol Device:Opamp_Dual_Generic
- added U?: STM32F103C8T6, Package_QFP:LQFP-48_7x7mm_P0.5mm, symbol MCU_ST_STM32F1:STM32F103C8Tx
- added U?: 128x32 OLED, Connector_PinSocket_2.54mm:PinSocket_1x04_P2.54mm_Vertical, symbol Connector_Generic:Conn_01x04
- added Y?: 8M, Crystal:Crystal_SMD_HC49-SD, symbol Device:Crystal_Small
Connections:
- net at Q?.1 (G): now also Q?.3 (C), R?.2
- net Iron+: now reaches Q?.2 (D)
- net Iron+: now also J?.1 (Pin_1), R?.1
- net +15V: now reaches Q?.3 (S)
- net +15V: now also C?.1, J?.1, R?.1, R?.1, U?.2 (Vin)
- new net: C?.2, U?.1 (Boost)
- new net: C?.1, L?.1, U?.3 (SW)
- new net: R?.2, R?.2, U?.5 (FB)
- new net: R?.1, U?.6 (COMP)
- new net: R?.2, U?.7 (Enable)
- new net: C?.1, U?.8 (SS)
- new net: C?.2, R?.2
- new net: D?.1 (K), R?.2
- new net: D?.2 (A), R?.2
- new net: R?.2, U?.1 (K), U?.3 (+)
- new net: R?.1, RV?.1, U?.1
- new net: R?.2, RV?.3
- new net: R?.1, R?.2, U?.2 (-)
- new net: Q?.1 (B), R?.1
- new net: R?.1, U?.44 (BOOT0)
- new net: R?.1, U?.20 (PB2)
- new net: C?.1, R?.2, U?.5 (PD0), Y?.1
- new net: C?.1, R?.1, U?.6 (PD1), Y?.2
- new net +3V3: C?.2, C?.2, C?.2, C?.2, C?.2, C?.2, J?.1 (Pin_1), L?.2, R?.1, R?.1, U?.1 (VBAT), U?.2 (Pin_2), U?.24 (VDD), U?.36 (VDD), U?.48 (VDD), U?.8 (V+), U?.9 (VDDA)
- new net GND: C?.1, C?.1, C?.1, C?.1, C?.1, C?.1, C?.1, C?.1, C?.2, C?.2, C?.2, C?.2, J?.1 (Pin_1), J?.1 (Pin_1), J?.2, J?.2 (Pin_2), Q?.2 (E), R?.1, R?.1, R?.2, R?.2, U?.1 (Pin_1), U?.2 (A), U?.23 (VSS), U?.35 (VSS), U?.4 (GND), U?.4 (V-), U?.47 (VSS), U?.8 (VSSA)
- new net NRST: C?.2, J?.6 (Pin_6), U?.7 (NRST)
- new net PWM: R?.2
- new net SCL: U?.3 (Pin_3)
- new net SDA: U?.4 (Pin_4)
- new net SWDCLK: J?.4 (Pin_4), U?.37 (PA14)
- new net SWDIO: J?.3 (Pin_3), U?.34 (PA13)
- new net SWO: J?.5 (Pin_5), U?.39 (PB3)
- no-connect marks 0 -> 3
Other:
- note added: "https://gitee.com/Cai-Zi/STM32_T12_Controller"
- moved on the sheet: Q?

Commit message: hardware
Parts:
- J2, J3, J4: renamed from J?; PartNum (none) -> C3130
- J5: renamed from J?; footprint (none) -> Connector_PinHeader_1.27mm:PinHeader_2x03_P1.27mm_Vertical; PartNum (none) -> C3408
- R10: renamed from R?; value R_Small -> 10k
- R2, R4, R9: renamed from R?; value R_Small -> 1k
- R7: renamed from R?; value R_Small -> 51k
- gave numbers to parts that had none: 34
Connections:
- net TEMP_ADC: now reaches D1.2 (A), R4.2
- net at R4.1, RV1.1, U1.1: now also RV1.2
Other:
- moved on the sheet: C1, D1, R10, R2, R4, R7, R9, RV1, U1A, U1B, U1C, U3

Commit message: hardware
Parts:
- C1, C10, C11, C12, C13, C3, C4, C5, C7, C8, C9: footprint (none) -> Capacitor_SMD:C_0603_1608Metric
- D1: footprint (none) -> Diode_SMD:D_SMA; PartNum (none) -> C437199
- J1: footprint (none) -> KIGIT_Connector:DC-050_2.5x5.5mm_SMT; PartNum (none) -> *
- J2, J3, J4: footprint (none) -> ts100:Fuseholder_5x20mm_inline
- L1: footprint (none) -> ts100:Inductor_SMD_5x4.5mm; PartNum (none) -> C576569
- R1, R10, R11, R12, R13, R14, R2, R3, R4, R5, R6, R7, R8, R9: footprint (none) -> Resistor_SMD:R_0603_1608Metric
Changed lines of the file:
@@
 F 0 "J1" H 907 1275 50  0000 C CNN
 F 1 "Jack-DC" H 907 1184 50  0000 C CNN
-F 2 "" H 900 910 50  0001 C CNN
+F 2 "KIGIT_Connector:DC-050_2.5x5.5mm_SMT" H 900 910 50  0001 C CNN
 F 3 "~" H 900 910 50  0001 C CNN
+F 4 "*" H 850 950 50  0001 C CNN "PartNum"
 	1    850  950
 	1    0    0    -1
@@
 F 0 "R3" H 1159 1846 50  0000 L CNN
 F 1 "100k" H 1159 1755 50  0000 L CNN
-F 2 "" H 1100 1800 50  0001 C CNN
+F 2 "Resistor_SMD:R_0603_1608Metric" H 1100 1800 50  0001 C CNN
 F 3 "~" H 1100 1800 50  0001 C CNN
 	1    1100 1800
@@
 F 0 "L1" V 2850 1900 50  0000 L CNN
 F 1 "6.8u" V 2750 1850 50  0000 L CNN
-F 2 "" H 2650 1950 50  0001 C CNN
+F 2 "ts100:Inductor_SMD_5x4.5mm" H 2650 1950 50  0001 C CNN
 F 3 "~" H 2650 1950 50  0001 C CNN
+F 4 "C576569" H 2650 1950 50  0001 C CNN "PartNum"
 	1    2650 1950
 	0    -1   -1   0
@@
 F 0 "C3" H 1342 2446 50  0000 L CNN
 F 1 "0.1u" H 1342 2355 50  0000 L CNN
-F 2 "" H 1250 2400 50  0001 C CNN
+F 2 "Capacitor_SMD:C_0603_1608Metric" H 1250 2400 50  0001 C CNN
 F 3 "~" H 1250 2400 50  0001 C CNN
 	1    1250 2400
@@
 F 0 "C5" V 2021 1500 50  0000 C CNN
 F 1 "10n" V 2112 1500 50  0000 C CNN
-F 2 "" H 2250 1500 50  0001 C CNN
+F 2 "Capacitor_SMD:C_0603_1608Metric" H 2250 1500 50  0001 C CNN
 F 3 "~" H 2250 1500 50  0001 C CNN
 	1    2250 1500
@@
 F 0 "R11" V 2550 2100 50  0000 L CNN
 F 1 "31.25k" V 2750 2050 50  0000 L CNN
-F 2 "" H 2650 2150 50  0001 C CNN
+F 2 "Resistor_SMD:R_0603_1608Metric" H 2650 2150 50  0001 C CNN
 F 3 "~" H 2650 2150 50  0001 C CNN
 	1    2650 2150
@@
 F 0 "R8" H 2509 2546 50  0000 L CNN
 F 1 "10k" H 2509 2455 50  0000 L CNN
-F 2 "" H 2450 2500 50  0001 C CNN
+F 2 "Resistor_SMD:R_0603_1608Metric" H 2450 2500 50  0001 C CNN
 F 3 "~" H 2450 2500 50  0001 C CNN
 	1    2450 2500
@@
 F 0 "R6" H 2009 2646 50  0000 L CNN
 F 1 "10k" H 2009 2555 50  0000 L CNN
-F 2 "" H 1950 2600 50  0001 C CNN
+F 2 "Resistor_SMD:R_0603_1608Metric" H 1950 2600 50  0001 C CNN
 F 3 "~" H 1950 2600 50  0001 C CNN
 	1    1950 2600
@@
 F 0 "C4" H 1858 2804 50  0000 R CNN
 F 1 "2.2n" H 1858 2895 50  0000 R CNN
-F 2 "" H 1950 2850 50  0001 C CNN
+F 2 "Capacitor_SMD:C_0603_1608Metric" H 1950 2850 50  0001 C CNN
 F 3 "~" H 1950 2850 50  0001 C CNN
 	1    1950 2850
@@
 F 0 "R5" H 1609 3946 50  0000 L CNN
 F 1 "10k" H 1609 3855 50  0000 L CNN
-F 2 "" H 1550 3900 50  0001 C CNN
+F 2 "Resistor_SMD:R_0603_1608Metric" H 1550 3900 50  0001 C CNN
 F 3 "~" H 1550 3900 50  0001 C CNN
 	1    1550 3900
@@
 F 0 "R1" V 754 4550 50  0000 C CNN
 F 1 "1k" V 845 4550 50  0000 C CNN
-F 2 "" H 950 4550 50  0001 C CNN
+F 2 "Resistor_SMD:R_0603_1608Metric" H 950 4550 50  0001 C CNN
 F 3 "~" H 950 4550 50  0001 C CNN
 	1    950  4550
@@
 F 0 "J2" H 2680 4942 50  0000 L CNN
 F 1 "Iron+" H 2680 4851 50  0000 L CNN
-F 2 "" H 2600 4900 50  0001 C CNN
+F 2 "ts100:Fuseholder_5x20mm_inline" H 2600 4900 50  0001 C CNN
 F 3 "~" H 2600 4900 50  0001 C CNN
 F 4 "C3130" H 2600 4900 50  0001 C CNN "PartNum"
@@
 F 0 "J3" H 2680 5192 50  0000 L CNN
 F 1 "Iron-" H 2680 5101 50  0000 L CNN
-F 2 "" H 2600 5150 50  0001 C CNN
+F 2 "ts100:Fuseholder_5x20mm_inline" H 2600 5150 50  0001 C CNN
 F 3 "~" H 2600 5150 50  0001 C CNN
 F 4 "C3130" H 2600 5150 50  0001 C CNN "PartNum"
@@
 F 0 "J4" V 3064 4812 50  0000 R CNN
 F 1 "GND" V 2973 4812 50  0000 R CNN
-F 2 "" H 3100 4900 50  0001 C CNN
+F 2 "ts100:Fuseholder_5x20mm_inline" H 3100 4900 50  0001 C CNN
 F 3 "~" H 3100 4900 50  0001 C CNN
 F 4 "C3130" H 3100 4900 50  0001 C CNN "PartNum"
@@
 F 0 "R2" H 1009 5946 50  0000 L CNN
 F 1 "1k" H 1009 5855 50  0000 L CNN
-F 2 "" H 950 5900 50  0001 C CNN
+F 2 "Resistor_SMD:R_0603_1608Metric" H 950 5900 50  0001 C CNN
 F 3 "~" H 950 5900 50  0001 C CNN
 	1    950  5900
@@
 F 0 "D1" V 904 6268 50  0000 L CNN
 F 1 "1N5819" V 995 6268 50  0000 L CNN
-F 2 "" V 950 6200 50  0001 C CNN
+F 2 "Diode_SMD:D_SMA" V 950 6200 50  0001 C CNN
 F 3 "~" V 950 6200 50  0001 C CNN
+F 4 "C437199" H 950 6200 50  0001 C CNN "PartNum"
 	1    950  6200
 	0    1    1    0
@@
 F 0 "R4" V 954 6550 50  0000 C CNN
 F 1 "1k" V 1045 6550 50  0000 C CNN
-F 2 "" H 1150 6550 50  0001 C CNN
+F 2 "Resistor_SMD:R_0603_1608Metric" H 1150 6550 50  0001 C CNN
 F 3 "~" H 1150 6550 50  0001 C CNN
 	1    1150 6550
@@
 F 0 "R7" V 1904 6150 50  0000 C CNN
 F 1 "51k" V 1995 6150 50  0000 C CNN
-F 2 "" H 2100 6150 50  0001 C CNN
+F 2 "Resistor_SMD:R_0603_1608Metric" H 2100 6150 50  0001 C CNN
 F 3 "~" H 2100 6150 50  0001 C CNN
 	1    2100 6150
@@
 F 0 "R9" V 2254 6450 50  0000 C CNN
 F 1 "1k" V 2345 6450 50  0000 C CNN
-F 2 "" H 2450 6450 50  0001 C CNN
+F 2 "Resistor_SMD:R_0603_1608Metric" H 2450 6450 50  0001 C CNN
 F 3 "~" H 2450 6450 50  0001 C CNN
 	1    2450 6450
@@
 F 0 "R10" V 2550 6650 50  0000 C CNN
 F 1 "10k" V 2650 6650 50  0000 C CNN
-F 2 "" H 2450 6650 50  0001 C CNN
+F 2 "Resistor_SMD:R_0603_1608Metric" H 2450 6650 50  0001 C CNN
 F 3 "~" H 2450 6650 50  0001 C CNN
 	1    2450 6650
@@
 F 0 "C1" H 608 6954 50  0000 R CNN
 F 1 "0.1u" H 608 7045 50  0000 R CNN
-F 2 "" H 700 7000 50  0001 C CNN
+F 2 "Capacitor_SMD:C_0603_1608Metric" H 700 7000 50  0001 C CNN
 F 3 "~" H 700 7000 50  0001 C CNN
 	1    700  7000
@@
 F 0 "R13" V 6800 2300 50  0000 C CNN
 F 1 "10k" V 7000 2300 50  0000 C CNN
-F 2 "" H 6900 2300 50  0001 C CNN
+F 2 "Resistor_SMD:R_0603_1608Metric" H 6900 2300 50  0001 C CNN
 F 3 "~" H 6900 2300 50  0001 C CNN
 	1    6900 2300
@@
 F 0 "R12" H 5841 2354 50  0000 R CNN
 F 1 "1M" H 5841 2445 50  0000 R CNN
-F 2 "" H 5900 2400 50  0001 C CNN
+F 2 "Resistor_SMD:R_0603_1608Metric" H 5900 2400 50  0001 C CNN
 F 3 "~" H 5900 2400 50  0001 C CNN
 	1    5900 2400
@@
 F 0 "C7" V 5471 2200 50  0000 C CNN
 F 1 "22p" V 5562 2200 50  0000 C CNN
-F 2 "" H 5700 2200 50  0001 C CNN
+F 2 "Capacitor_SMD:C_0603_1608Metric" H 5700 2200 50  0001 C CNN
 F 3 "~" H 5700 2200 50  0001 C CNN
 	1    5700 2200
@@
 F 0 "C8" V 5471 2600 50  0000 C CNN
 F 1 "22p" V 5562 2600 50  0000 C CNN
-F 2 "" H 5700 2600 50  0001 C CNN
+F 2 "Capacitor_SMD:C_0603_1608Metric" H 5700 2600 50  0001 C CNN
 F 3 "~" H 5700 2600 50  0001 C CNN
 	1    5700 2600
@@
 F 0 "C10" H 7592 1396 50  0000 L CNN
 F 1 "0.1u" H 7592 1305 50  0000 L CNN
-F 2 "" H 7500 1350 50  0001 C CNN
+F 2 "Capacitor_SMD:C_0603_1608Metric" H 7500 1350 50  0001 C CNN
 F 3 "~" H 7500 1350 50  0001 C CNN
 	1    7500 1350
@@
 F 0 "C11" H 7892 1396 50  0000 L CNN
 F 1 "0.1u" H 7892 1305 50  0000 L CNN
-F 2 "" H 7800 1350 50  0001 C CNN
+F 2 "Capacitor_SMD:C_0603_1608Metric" H 7800 1350 50  0001 C CNN
 F 3 "~" H 7800 1350 50  0001 C CNN
 	1    7800 1350
@@
 F 0 "C12" H 8192 1396 50  0000 L CNN
 F 1 "0.1u" H 8192 1305 50  0000 L CNN
-F 2 "" H 8100 1350 50  0001 C CNN
+F 2 "Capacitor_SMD:C_0603_1608Metric" H 8100 1350 50  0001 C CNN
 F 3 "~" H 8100 1350 50  0001 C CNN
 	1    8100 1350
@@
 F 0 "C13" H 8492 1396 50  0000 L CNN
 F 1 "0.1u" H 8492 1305 50  0000 L CNN
-F 2 "" H 8400 1350 50  0001 C CNN
+F 2 "Capacitor_SMD:C_0603_1608Metric" H 8400 1350 50  0001 C CNN
 F 3 "~" H 8400 1350 50  0001 C CNN
 	1    8400 1350
@@
 F 0 "R14" V 6704 3400 50  0000 C CNN
 F 1 "10k" V 6795 3400 50  0000 C CNN
-F 2 "" H 6900 3400 50  0001 C CNN
+F 2 "Resistor_SMD:R_0603_1608Metric" H 6900 3400 50  0001 C CNN
 F 3 "~" H 6900 3400 50  0001 C CNN
 	1    6900 3400
@@
 F 0 "C9" H 6792 1896 50  0000 L CNN
 F 1 "0.1u" H 6792 1805 50  0000 L CNN
-F 2 "" H 6700 1850 50  0001 C CNN
+F 2 "Capacitor_SMD:C_0603_1608Metric" H 6700 1850 50  0001 C CNN
 F 3 "~" H 6700 1850 50  0001 C CNN
 	1    6700 1850

Commit message: hardware
Parts:
- added S?: SW18010P, Capacitor_THT:C_Radial_D5.0mm_H5.0mm_P2.00mm, symbol KIGIT_Sensor:SW18010P
- added SW? (x2): SW_Push, symbol Switch:SW_Push
- J5: footprint Connector_PinHeader_1.27mm:PinHeader_2x03_P1.27mm_Vertical -> Connector_PinHeader_1.27mm:PinHeader_1x06_P1.27mm_Vertical; symbol Connector_Generic:Conn_02x03_Odd_Even -> Connector_Generic:Conn_01x06
Connections:
- net +3V3: now also J5.2 (Pin_2); no longer J5.1 (Pin_1)
- net GND: no longer J5.2 (Pin_2)
- net NRST: no longer J5.6 (Pin_6)
- net SWDCLK: no longer J5.4 (Pin_4)
- net SWO: now also J5.4 (Pin_4); no longer J5.5 (Pin_5)
Other:
- moved on the sheet: C10, C11, C12, C13, C7, C8, C9, J5, R12, R13, R14, U4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

Commit message: pcb
Parts:
- U3: PartNum (none) -> C140852
Connections:
- net PWM: now also U5.10 (PA0)
- net SCL: now also U5.42 (PB6)
- net SDA: now also U5.43 (PB7)
- net TEMP_ADC: now also U5.11 (PA1)
- no-connect marks 3 -> 30
Other:
- moved on the sheet: S?
Changed lines of the file:
@@
 F 2 "Diode_THT:D_DO-41_SOD81_P7.62mm_Horizontal" H 2200 6850 50  0001 C CIN
 F 3 "http://www.ti.com/lit/ds/symlink/lm4040-n.pdf" H 2200 7050 50  0001 C CIN
+F 4 "C140852" H 2200 7050 50  0001 C CNN "PartNum"
 	1    2200 7050
 	0    -1   -1   0
@@
 L KIGIT_Sensor:SW18010P S?
 U 1 1 615237D9
-P 8750 4800
-F 0 "S?" H 9208 4813 50  0000 L CNN
-F 1 "SW18010P" H 9208 4722 50  0000 L CNN
-F 2 "Capacitor_THT:C_Radial_D5.0mm_H5.0mm_P2.00mm" H 8750 5150 50  0001 C CNN
-F 3 "" H 8750 5150 50  0001 C CNN
-F 4 "C2681585" H 8750 4800 50  0001 C CNN "PartNum"
-	1    8750 4800
-	1    0    0    -1
-$EndComp
+P 9350 4400
+F 0 "S?" H 9808 4413 50  0000 L CNN
+F 1 "SW18010P" H 9808 4322 50  0000 L CNN
+F 2 "Capacitor_THT:C_Radial_D5.0mm_H5.0mm_P2.00mm" H 9350 4750 50  0001 C CNN
+F 3 "" H 9350 4750 50  0001 C CNN
+F 4 "C2681585" H 9350 4400 50  0001 C CNN "PartNum"
+	1    9350 4400
+	1    0    0    -1
+$EndComp
+Text Label 5000 3500 0    50   ~ 0
+SCL
+Text Label 5000 3600 0    50   ~ 0
+SDA
+Text Label 7100 2900 0    50   ~ 0
+PWM
+Text Label 7100 3000 0    50   ~ 0
+TEMP_ADC
+Wire Wire Line
+	5450 3500 5000 3500
+Wire Wire Line
+	5450 3600 5000 3600
+Wire Wire Line
+	6750 2900 7100 2900
+Wire Wire Line
+	6750 3000 7100 3000
+NoConn ~ 5450 2500
+NoConn ~ 5450 2600
+NoConn ~ 5450 2700
+NoConn ~ 5450 2900
+NoConn ~ 5450 3000
+NoConn ~ 5450 3300
+NoConn ~ 5450 3400
+NoConn ~ 5450 3700
+NoConn ~ 5450 3800
+NoConn ~ 5450 3900
+NoConn ~ 5450 4000
+NoConn ~ 5450 4100
+NoConn ~ 5450 4200
+NoConn ~ 5450 4300
+NoConn ~ 5450 4400
+NoConn ~ 6750 4400
+NoConn ~ 6750 4100
+NoConn ~ 6750 4000
+NoConn ~ 6750 3900
+NoConn ~ 6750 3800
+NoConn ~ 6750 3700
+NoConn ~ 6750 3600
+NoConn ~ 6750 3500
+NoConn ~ 6750 3400
+NoConn ~ 6750 3300
+NoConn ~ 6750 3200
+NoConn ~ 6750 3100
+$Comp
+L power:PWR_FLAG #FLG0103
+U 1 1 615821AF
+P 3200 1950
+F 0 "#FLG0103" H 3200 2025 50  0001 C CNN
+F 1 "PWR_FLAG" H 3200 2123 50  0000 C CNN
+F 2 "" H 3200 1950 50  0001 C CNN
+F 3 "~" H 3200 1950 50  0001 C CNN
+	1    3200 1950
+	1    0    0    -1
+$EndComp
+Wire Wire Line
+	2850 1950 3200 1950
 $EndSCHEMATC

Commit message: hardware
Parts:
- gave numbers to parts that had none: 2
Connections:
- net GND: now also S?.1, SW1.2, SW2.2
- net WAK_UP: now reaches U5.21 (PB10)
- net WAK_UP: now also S?.2
- net KEY1: now reaches U5.45 (PB8)
- net KEY1: now also SW1.1
- net KEY2: now reaches U5.46 (PB9)
- net KEY2: now also SW2.1
- no-connect marks 30 -> 27
Other:
- moved on the sheet: SW1, SW2
Changed lines of the file:
@@
 Connection ~ 950  6550
 $Comp
-L Switch:SW_Push SW?
+L Switch:SW_Push SW1
 U 1 1 6151F8F6
-P 9350 3450
-F 0 "SW?" H 9350 3735 50  0000 C CNN
-F 1 "SW_Push" H 9350 3644 50  0000 C CNN
-F 2 "" H 9350 3650 50  0001 C CNN
-F 3 "~" H 9350 3650 50  0001 C CNN
-F 4 "C319392" H 9350 3450 50  0001 C CNN "PartNum"
-	1    9350 3450
+P 9300 3200
+F 0 "SW1" H 9300 3485 50  0000 C CNN
+F 1 "SW_Push" H 9300 3394 50  0000 C CNN
+F 2 "" H 9300 3400 50  0001 C CNN
+F 3 "~" H 9300 3400 50  0001 C CNN
+F 4 "C319392" H 9300 3200 50  0001 C CNN "PartNum"
+	1    9300 3200
 	1    0    0    -1
 $EndComp
 $Comp
-L Switch:SW_Push SW?
+L Switch:SW_Push SW2
 U 1 1 615205A5
-P 9350 3900
-F 0 "SW?" H 9350 4185 50  0000 C CNN
-F 1 "SW_Push" H 9350 4094 50  0000 C CNN
-F 2 "" H 9350 4100 50  0001 C CNN
-F 3 "~" H 9350 4100 50  0001 C CNN
-F 4 "C319392" H 9350 3900 50  0001 C CNN "PartNum"
-	1    9350 3900
+P 9300 3650
+F 0 "SW2" H 9300 3935 50  0000 C CNN
+F 1 "SW_Push" H 9300 3844 50  0000 C CNN
+F 2 "" H 9300 3850 50  0001 C CNN
+F 3 "~" H 9300 3850 50  0001 C CNN
+F 4 "C319392" H 9300 3650 50  0001 C CNN "PartNum"
+	1    9300 3650
 	1    0    0    -1
 $EndComp
@@
 NoConn ~ 5450 3300
 NoConn ~ 5450 3400
-NoConn ~ 5450 3700
-NoConn ~ 5450 3800
-NoConn ~ 5450 3900
 NoConn ~ 5450 4000
 NoConn ~ 5450 4100
@@
 Wire Wire Line
 	2850 1950 3200 1950
+$Comp
+L power:GND #PWR?
+U 1 1 6161C01C
+P 9850 3300
+F 0 "#PWR?" H 9850 3050 50  0001 C CNN
+F 1 "GND" H 9855 3127 50  0000 C CNN
+F 2 "" H 9850 3300 50  0001 C CNN
+F 3 "" H 9850 3300 50  0001 C CNN
+	1    9850 3300
+	1    0    0    -1
+$EndComp
+$Comp
+L power:GND #PWR?
+U 1 1 61621F30
+P 9850 3750
+F 0 "#PWR?" H 9850 3500 50  0001 C CNN
+F 1 "GND" H 9855 3577 50  0000 C CNN
+F 2 "" H 9850 3750 50  0001 C CNN
+F 3 "" H 9850 3750 50  0001 C CNN
+	1    9850 3750
+	1    0    0    -1
+$EndComp
+Wire Wire Line
+	9500 3200 9850 3200
+Wire Wire Line
+	9850 3200 9850 3300
+Wire Wire Line
+	9500 3650 9850 3650
+Wire Wire Line
+	9850 3650 9850 3750
+Wire Wire Line
+	9100 3650 8850 3650
+Wire Wire Line
+	9100 3200 8850 3200
+Text Label 8850 3200 0    50   ~ 0
+KEY1
+Text Label 8850 3650 0    50   ~ 0
+KEY2
+$Comp
+L power:GND #PWR?
+U 1 1 61643B2A
+P 9750 4650
+F 0 "#PWR?" H 9750 4400 50  0001 C CNN
+F 1 "GND" H 9755 4477 50  0000 C CNN
+F 2 "" H 9750 4650 50  0001 C CNN
+F 3 "" H 9750 4650 50  0001 C CNN
+	1    9750 4650
+	1    0    0    -1
+$EndComp
+Text Label 8550 4650 0    50   ~ 0
+WAK_UP
+Wire Wire Line
+	8950 4650 8550 4650
+Text Label 5000 3700 0    50   ~ 0
+KEY1
+Text Label 5000 3800 0    50   ~ 0
+KEY2
+Text Label 5000 3900 0    50   ~ 0
+WAK_UP
+Wire Wire Line
+	5450 3700 5000 3700
+Wire Wire Line
+	5000 3800 5450 3800
+Wire Wire Line
+	5450 3900 5000 3900
 $EndSCHEMATC

Commit message: pcb
Parts:
- SW1, SW2: footprint (none) -> ts100:SMD,4.6x1.82x3.5mm
- gave numbers to parts that had none: 1
Connections:
- net GND: now also J5.1 (Pin_1)
- net NRST: now also J5.6 (Pin_6)
- net SWDCLK: now also J5.5 (Pin_5)
Changed lines of the file:
@@
 U 1 1 615587B3
 P 9300 1350
-F 0 "J5" H 9350 1667 50  0000 C CNN
-F 1 "SWD" H 9350 1576 50  0000 C CNN
+F 0 "J5" H 9300 1650 50  0000 C CNN
+F 1 "SWD" H 9300 950 50  0000 C CNN
 F 2 "Connector_PinHeader_1.27mm:PinHeader_1x06_P1.27mm_Vertical" H 9300 1350 50  0001 C CNN
 F 3 "~" H 9300 1350 50  0001 C CNN
@@
 	-1   0    0    1
 $EndComp
-Text Label 8850 1450 0    50   ~ 0
+Text Label 8800 1450 0    50   ~ 0
 SWO
-Text Label 9700 1350 0    50   ~ 0
+Text Label 8800 1550 0    50   ~ 0
 SWDCLK
-Text Label 8850 1350 0    50   ~ 0
+Text Label 8800 1350 0    50   ~ 0
 SWDIO
-Text Label 9700 1450 0    50   ~ 0
+Text Label 8800 1650 0    50   ~ 0
 NRST
-Wire Wire Line
-	9100 1350 8850 1350
-Wire Wire Line
-	8850 1450 9100 1450
-Wire Wire Line
-	9600 1350 9700 1350
-Wire Wire Line
-	9600 1450 9700 1450
 $Comp
 L power:GND #PWR0125
 U 1 1 6157108F
-P 9800 1250
-F 0 "#PWR0125" H 9800 1000 50  0001 C CNN
-F 1 "GND" H 9805 1077 50  0000 C CNN
-F 2 "" H 9800 1250 50  0001 C CNN
-F 3 "" H 9800 1250 50  0001 C CNN
-	1    9800 1250
+P 9050 1000
+F 0 "#PWR0125" H 9050 750 50  0001 C CNN
+F 1 "GND" H 9055 827 50  0000 C CNN
+F 2 "" H 9050 1000 50  0001 C CNN
+F 3 "" H 9050 1000 50  0001 C CNN
+	1    9050 1000
 	-1   0    0    1
 $EndComp
@@
 Wire Wire Line
 	8900 1250 9100 1250
-Wire Wire Line
-	9600 1250 9800 1250
 $Comp
 L Connector_Generic:Conn_01x04 U4
@@
 F 0 "SW1" H 9300 3485 50  0000 C CNN
 F 1 "SW_Push" H 9300 3394 50  0000 C CNN
-F 2 "" H 9300 3400 50  0001 C CNN
+F 2 "ts100:SMD,4.6x1.82x3.5mm" H 9300 3400 50  0001 C CNN
 F 3 "~" H 9300 3400 50  0001 C CNN
 F 4 "C319392" H 9300 3200 50  0001 C CNN "PartNum"
@@
 F 0 "SW2" H 9300 3935 50  0000 C CNN
 F 1 "SW_Push" H 9300 3844 50  0000 C CNN
-F 2 "" H 9300 3850 50  0001 C CNN
+F 2 "ts100:SMD,4.6x1.82x3.5mm" H 9300 3850 50  0001 C CNN
 F 3 "~" H 9300 3850 50  0001 C CNN
 F 4 "C319392" H 9300 3650 50  0001 C CNN "PartNum"
@@
 $EndComp
 $Comp
-L KIGIT_Sensor:SW18010P S?
+L KIGIT_Sensor:SW18010P S1
 U 1 1 615237D9
 P 9350 4400
-F 0 "S?" H 9808 4413 50  0000 L CNN
+F 0 "S1" H 9808 4413 50  0000 L CNN
 F 1 "SW18010P" H 9808 4322 50  0000 L CNN
 F 2 "Capacitor_THT:C_Radial_D5.0mm_H5.0mm_P2.00mm" H 9350 4750 50  0001 C CNN
@@
 	2850 1950 3200 1950
 $Comp
-L power:GND #PWR?
+L power:GND #PWR0129
 U 1 1 6161C01C
 P 9850 3300
-F 0 "#PWR?" H 9850 3050 50  0001 C CNN
+F 0 "#PWR0129" H 9850 3050 50  0001 C CNN
 F 1 "GND" H 9855 3127 50  0000 C CNN
 F 2 "" H 9850 3300 50  0001 C CNN
@@
 $EndComp
 $Comp
-L power:GND #PWR?
+L power:GND #PWR0130
 U 1 1 61621F30
 P 9850 3750
-F 0 "#PWR?" H 9850 3500 50  0001 C CNN
+F 0 "#PWR0130" H 9850 3500 50  0001 C CNN
 F 1 "GND" H 9855 3577 50  0000 C CNN
 F 2 "" H 9850 3750 50  0001 C CNN
@@
 KEY2
 $Comp
-L power:GND #PWR?
+L power:GND #PWR0131
 U 1 1 61643B2A
 P 9750 4650
-F 0 "#PWR?" H 9750 4400 50  0001 C CNN
+F 0 "#PWR0131" H 9750 4400 50  0001 C CNN
 F 1 "GND" H 9755 4477 50  0000 C CNN
 F 2 "" H 9750 4650 50  0001 C CNN
@@
 Wire Wire Line
 	5450 3900 5000 3900
+Wire Wire Line
+	9050 1000 9050 1150
+Wire Wire Line
+	9050 1150 9100 1150
+Wire Wire Line
+	8800 1350 9100 1350
+Wire Wire Line
+	8800 1450 9100 1450
+Wire Wire Line
+	9100 1550 8800 1550
+Wire Wire Line
+	9100 1650 8800 1650
 $EndSCHEMATC
