File: Hardware/ts100.kicad_sch (KiCad schematic)
At the start: 38 parts, among them J1 Jack-DC, J2 Iron+, J3 Iron-, J4 GND, J5 Debug, K1 TMP_UP, K2 TMP_DOWN, Q1 2SC3356, Q2 IRF4905STRLPBF, U1 LM358G-S08-R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

Commit message: 核对封装
Parts:
- C8: footprint Capacitor_SMD:C_0603_1608Metric -> Capacitor_SMD:C_0402_1005Metric
- C9: PartNum (none) -> C107372
- FB1: PartNum (none) -> C21286
- J1: PartNum * -> C720583
- R6, R7: footprint Resistor_SMD:R_0603_1608Metric -> Resistor_SMD:R_0402_1005Metric
Connections:
- net SWIM: now also U3.18 (PD1)
- no-connect marks 11 -> 9
Changed lines of the file:
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@@
   (junction (at 15.24 48.26) (diameter 0) (color 0 0 0 0)
   )
-  (no_connect (at 100.965 72.39))
   (no_connect (at 144.78 92.71))
   (no_connect (at 144.78 87.63))
   (no_connect (at 175.26 80.01))
   (no_connect (at 59.69 189.23))
-  (no_connect (at 175.26 74.93))
   (no_connect (at 59.69 184.15))
   (no_connect (at 144.78 82.55))
@@
     (stroke (width 0) (type default) (color 0 0 0 0))
   )
+  (wire (pts (xy 175.26 74.93) (xy 179.07 74.93))
+    (stroke (width 0) (type default) (color 0 0 0 0))
+  )
   (wire (pts (xy 52.07 55.88) (xy 52.07 66.04))
     (stroke (width 0) (type default) (color 0 0 0 0))
@@
   )
   (label "KEY1" (at 179.07 82.55 0)
+    (effects (font (size 1.27 1.27)) (justify left bottom))
+  )
+  (label "SWIM" (at 179.07 74.93 0)
     (effects (font (size 1.27 1.27)) (justify left bottom))
   )
@@
       (effects (font (size 1.27 1.27)) hide)
     )
-    (property "PartNum" "*" (id 4) (at 21.59 24.13 0)
+    (property "PartNum" "C720583" (id 4) (at 21.59 24.13 0)
       (effects (font (size 1.27 1.27)) hide)
     )
@@
       (effects (font (size 1.27 1.27)) (justify left))
     )
-    (property "Footprint" "Resistor_SMD:R_0603_1608Metric" (id 2) (at 72.39 69.85 0)
+    (property "Footprint" "Resistor_SMD:R_0402_1005Metric" (id 2) (at 72.39 69.85 0)
       (effects (font (size 1.27 1.27)) hide)
     )
@@
       (effects (font (size 1.27 1.27)) (justify left))
     )
-    (property "Footprint" "Resistor_SMD:R_0603_1608Metric" (id 2) (at 72.39 62.23 0)
+    (property "Footprint" "Resistor_SMD:R_0402_1005Metric" (id 2) (at 72.39 62.23 0)
       (effects (font (size 1.27 1.27)) hide)
     )
@@
       (effects (font (size 1.27 1.27)) hide)
     )
+    (property "PartNum" "C21286" (id 4) (at 36.195 21.59 0)
+      (effects (font (size 1.27 1.27)) hide)
+    )
     (pin "1")
     (pin "2")
@@
     )
     (property "Datasheet" "~" (id 3) (at 134.62 104.775 0)
+      (effects (font (size 1.27 1.27)) hide)
+    )
+    (property "PartNum" "C107372" (id 4) (at 134.62 104.775 0)
       (effects (font (size 1.27 1.27)) hide)
     )
@@
       (effects (font (size 1.27 1.27)) (justify left))
     )
-    (property "Footprint" "Capacitor_SMD:C_0603_1608Metric" (id 2) (at 134.62 91.44 0)
+    (property "Footprint" "Capacitor_SMD:C_0402_1005Metric" (id 2) (at 134.62 91.44 0)
       (effects (font (size 1.27 1.27)) hide)
     )
@@
     )
     (path "/91d4048c-e95f-4533-ad0d-93a5a478aa95"
-      (reference "C8") (unit 1) (value "0.1u") (footprint "Capacitor_SMD:C_0603_1608Metric")
+      (reference "C8") (unit 1) (value "0.1u") (footprint "Capacitor_SMD:C_0402_1005Metric")
     )
     (path "/16f219d5-8df5-4f96-b872-6d28f60997d4"
@@
     )
     (path "/00000000-0000-0000-0000-000061d3ec03"
-      (reference "R6") (unit 1) (value "68k 1%") (footprint "Resistor_SMD:R_0603_1608Metric")
+      (reference "R6") (unit 1) (value "68k 1%") (footprint "Resistor_SMD:R_0402_1005Metric")
     )
     (path "/00000000-0000-0000-0000-000061d3dbc2"
-      (reference "R7") (unit 1) (value "13k 1%") (footprint "Resistor_SMD:R_0603_1608Metric")
+      (reference "R7") (unit 1) (value "13k 1%") (footprint "Resistor_SMD:R_0402_1005Metric")
     )
     (path "/00000000-0000-0000-0000-000062118b2e"

Commit message: 修改封装
Parts:
- J1: footprint KIGIT_Connectors:DC-050_2.5x5.5mm_SMT -> Connector_BarrelJack:BarrelJack_CLIFF_FC681465S_SMT_Horizontal
Changed lines of the file:
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@@
   (junction (at 52.07 92.71) (diameter 0) (color 0 0 0 0)
   )
-  (junction (at -66.04 191.77) (diameter 0) (color 0 0 0 0)
-  )
   (junction (at 52.07 157.48) (diameter 0) (color 0 0 0 0)
   )
   (junction (at 59.69 52.07) (diameter 0) (color 0 0 0 0)
+  )
+  (junction (at 74.295 52.07) (diameter 0) (color 0 0 0 0)
   )
   (junction (at 33.02 26.67) (diameter 0) (color 0 0 0 0)
@@
     (stroke (width 0) (type default) (color 0 0 0 0))
   )
+  (wire (pts (xy 74.295 49.53) (xy 74.295 52.07))
+    (stroke (width 0) (type default) (color 0 0 0 0))
+  )
   (wire (pts (xy 15.24 46.99) (xy 15.24 48.26))
     (stroke (width 0) (type default) (color 0 0 0 0))
@@
     (stroke (width 0) (type default) (color 0 0 0 0))
   )
-  (wire (pts (xy -68.58 191.77) (xy -66.04 191.77))
+  (wire (pts (xy 74.295 52.07) (xy 76.2 52.07))
     (stroke (width 0) (type default) (color 0 0 0 0))
   )
@@
     (stroke (width 0) (type default) (color 0 0 0 0))
   )
-  (wire (pts (xy -66.04 191.77) (xy -63.5 191.77))
-    (stroke (width 0) (type default) (color 0 0 0 0))
-  )
   (wire (pts (xy 238.125 107.315) (xy 238.125 109.855))
     (stroke (width 0) (type default) (color 0 0 0 0))
@@
     (stroke (width 0) (type default) (color 0 0 0 0))
   )
-  (wire (pts (xy 72.39 52.07) (xy 76.2 52.07))
+  (wire (pts (xy 72.39 52.07) (xy 74.295 52.07))
     (stroke (width 0) (type default) (color 0 0 0 0))
   )
@@
   )
   (wire (pts (xy 52.07 124.46) (xy 60.96 124.46))
-    (stroke (width 0) (type default) (color 0 0 0 0))
-  )
-  (wire (pts (xy -66.04 173.355) (xy -66.04 191.77))
     (stroke (width 0) (type default) (color 0 0 0 0))
   )
@@
     (effects (font (size 1.27 1.27)) (justify left bottom))
   )
-  (label "TEMP_ADC" (at -33.02 234.315 0)
-    (effects (font (size 1.27 1.27)) (justify left bottom))
-  )
   (label "HSE_IN" (at 135.89 64.77 0)
     (effects (font (size 1.27 1.27)) (justify left bottom))
@@
     (property "Reference" "J1" (id 0) (at 23.0378 15.875 0))
     (property "Value" "Jack-DC" (id 1) (at 23.0378 18.1864 0))
-    (property "Footprint" "KIGIT_Connectors:DC-050_2.5x5.5mm_SMT" (id 2) (at 22.86 25.146 0)
+    (property "Footprint" "Connector_BarrelJack:BarrelJack_CLIFF_FC681465S_SMT_Horizontal" (id 2) (at 22.86 25.146 0)
       (effects (font (size 1.27 1.27)) hide)
     )
@@
     (pin "2")
   )
+  (symbol (lib_id "power:PWR_FLAG") (at 74.295 49.53 0) (unit 1)
+    (in_bom yes) (on_board yes)
+    (property "Reference" "#FLG0101" (id 0) (at 74.295 47.625 0)
+      (effects (font (size 1.27 1.27)) hide)
+    )
+    (property "Value" "PWR_FLAG" (id 1) (at 74.295 45.1358 0))
+    (property "Footprint" "" (id 2) (at 74.295 49.53 0)
+      (effects (font (size 1.27 1.27)) hide)
+    )
+    (property "Datasheet" "~" (id 3) (at 74.295 49.53 0)
+      (effects (font (size 1.27 1.27)) hide)
+    )
+    (pin "1")
+  )
   (symbol (lib_id "power:+5V") (at 208.28 68.58 0) (unit 1)
     (in_bom yes) (on_board yes) (fields_autoplaced)
@@
       (reference "#FLG02") (unit 1) (value "PWR_FLAG") (footprint "")
     )
+    (path "/e8c057d7-6bb8-4489-9655-d10ccc0dc3e3"
+      (reference "#FLG0101") (unit 1) (value "PWR_FLAG") (footprint "")
+    )
     (path "/00000000-0000-0000-0000-000061d6a8b9"
       (reference "#PWR01") (unit 1) (value "+19V") (footprint "")
@@
     )
     (path "/00000000-0000-0000-0000-000061435429"
-      (reference "J1") (unit 1) (value "Jack-DC") (footprint "KIGIT_Connectors:DC-050_2.5x5.5mm_SMT")
+      (reference "J1") (unit 1) (value "Jack-DC") (footprint "Connector_BarrelJack:BarrelJack_CLIFF_FC681465S_SMT_Horizontal")
     )
     (path "/00000000-0000-0000-0000-000061478e68"
